File: kicad/_autosave-solderbit-gamepad.kicad_pcb (KiCad board)
At the start: 2 copper layers, 33 parts, among them SW7 SW_Push, SW8 SW_Push, U1 Shift_Register_74HC165D

Commit message: New updates on the PCB, libraries, and other
Parts:
- C1, C2, C3, C4, C5, C6: footprint Capacitor_SMD:C_1206_3216Metric_Pad1.33x1.80mm_HandSolder -> Solderbit_Gamepad:1206_Capacitor
- D1, D2, D3, D4, D5: value NeoPixel_WS2812B -> WS2812B
- R1, R2, R3, R4, R5, R6, R7, R8, R9: footprint Resistor_SMD:R_1206_3216Metric_Pad1.30x1.75mm_HandSolder -> Solderbit_Gamepad:1206_Resistor
- U1: value Shift_Register_74HC165D -> Val**
- moved D1 40.8 mm to (128.4, 52.0), turned to 0 degrees
- moved D5 24.6 mm to (88.4, 52.0), turned to 0 degrees
- moved D2 24.4 mm to (118.4, 52.0), turned to 0 degrees
- moved C6 15.1 mm to (127.8, 60.0)
- moved C5 14.9 mm to (121.2, 60.0)
- moved C4 14.8 mm to (114.8, 60.0)
- moved S5 12.0 mm to (145.0, 55.0)
- moved S6 12.0 mm to (160.0, 45.0)
- moved C1 9.68 mm to (105.0, 76.7), turned to -90 degrees
- moved D4 8.29 mm to (98.4, 52.0), turned to 0 degrees
- moved D3 8.09 mm to (108.4, 52.0), turned to 0 degrees
- moved R5 6.83 mm to (155.0, 68.3)
- moved REF1 5.65 mm to (108.6, 35.0)
- moved C3 5.05 mm to (98.3, 60.0)
- moved R6 5.00 mm to (160.0, 68.3)
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Other:
- board text added: "v0.5"
- board text removed: "v1.4"
