File: kicad/_autosave-solderbit-gamepad.kicad_sch (KiCad schematic)
At the start: 33 parts, among them SW7 SW_Push, SW8 SW_Push, U1 Shift_Register_74HC165D

Commit message: New updates on the PCB, libraries, and other
Parts:
- removed G2: ~, Solderbit_Gamepad:Lancaster_Cityscape, symbol Solderbit_Gamepad:Lancaster_Cityscape_Image
Changed lines of the file:
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@@
-	)
-	(symbol
-		(lib_id "Solderbit_Gamepad:Lancaster_Cityscape_Image")
-		(at 134.62 165.1 0)
-		(unit 1)
-		(exclude_from_sim no)
-		(in_bom no)
-		(on_board yes)
-		(dnp no)
-		(fields_autoplaced yes)
-		(property "Reference" "G2"
-			(at 134.62 165.1 0)
-			(effects
-				(font
-					(size 1.27 1.27)
-				)
-				(hide yes)
-			)
-		)
-		(property "Value" "~"
-			(at 134.62 165.1 0)
-			(effects
-				(font
-					(size 1.27 1.27)
-				)
-				(hide yes)
-			)
-		)
-		(property "Footprint" "Solderbit_Gamepad:Lancaster_Cityscape"
-			(at 134.62 162.814 0)
-			(effects
-				(font
-					(size 1.27 1.27)
-				)
-				(hide yes)
-			)
-		)
-		(property "Datasheet" ""
-			(at 134.62 165.1 0)
-			(effects
-				(font
-					(size 1.27 1.27)
-				)
-				(hide yes)
-			)
-		)
-		(property "Description" ""
-			(at 134.62 165.1 0)
-			(effects
-				(font
-					(size 1.27 1.27)
-				)
-				(hide yes)
-			)
-		)
-		(instances
-			(project "solderbit-gamepad"
-				(path "/5cb26b28-0a45-4802-97bd-4f21bb092ec3"
-					(reference "G2")
-					(unit 1)
-				)
-			)
-		)
 	)
 	(symbol
@@
 	(symbol
 		(lib_id "Solderbit_Gamepad:Devices-Lab_Logo_Placeholder")
-		(at 113.03 165.1 0)
+		(at 125.73 165.1 0)
 		(unit 1)
 		(exclude_from_sim no)
@@
 		(fields_autoplaced yes)
 		(property "Reference" "G1"
-			(at 108.204 165.1 0)
+			(at 120.904 165.1 0)
 			(effects
 				(font
@@
 		)
 		(property "Value" "~"
-			(at 113.03 165.1 0)
+			(at 125.73 165.1 0)
 			(effects
 				(font
@@
 		)
 		(property "Footprint" "Solderbit_Gamepad:Devices-Lab_Logo"
-			(at 113.03 165.1 0)
-			(effects
-				(font
-					(size 1.27 1.27)
-				)
-				(hide yes)
-			)
-		)
-		(property "Datasheet" ""
-			(at 113.03 165.1 0)
+			(at 125.73 165.1 0)
+			(effects
+				(font
+					(size 1.27 1.27)
+				)
+				(hide yes)
+			)
+		)
+		(property "Datasheet" ""
+			(at 125.73 165.1 0)
 			(effects
 				(font
@@
 		)
 		(property "Description" ""
-			(at 113.03 165.1 0)
+			(at 125.73 165.1 0)
 			(effects
 				(font
@@
 	(symbol
 		(lib_id "Solderbit_Gamepad:Key_Chain_Hole")
-		(at 154.94 166.37 0)
+		(at 148.59 167.64 0)
 		(unit 1)
 		(exclude_from_sim no)
@@
 		(fields_autoplaced yes)
 		(property "Reference" "G3"
-			(at 154.94 166.37 0)
+			(at 148.59 167.64 0)
 			(effects
 				(font
@@
 		)
 		(property "Value" "~"
-			(at 154.94 166.37 0)
+			(at 148.59 167.64 0)
 			(effects
 				(font
@@
 		)
 		(property "Footprint" "Solderbit_Gamepad:Key_Chain_Hole"
-			(at 154.94 166.37 0)
-			(effects
-				(font
-					(size 1.27 1.27)
-				)
-				(hide yes)
-			)
-		)
-		(property "Datasheet" ""
-			(at 154.94 166.37 0)
+			(at 148.59 167.64 0)
+			(effects
+				(font
+					(size 1.27 1.27)
+				)
+				(hide yes)
+			)
+		)
+		(property "Datasheet" ""
+			(at 148.59 167.64 0)
 			(effects
 				(font
@@
 		)
 		(property "Description" ""
-			(at 154.94 166.37 0)
-			(effects
-				(font
+			(at 148.59 167.64 0)
+			(effects
+				(font
