File: solderbit-gamepad-v0.1/solderbit-gamepad-v0.1.kicad_sch (KiCad schematic)
At the start: 23 parts, among them U1 74HC165D_653

Commit message: Begin version 0.7, and new spreadsheet
Other:
- company: Aron Eggens -> Lancaster University
- title: Micro:bit SMT soldering kit (basic) -> solder:bit Gamepad
